Commit message: different jont condfigurations

File: human_model_gazebo/urdf/human.xacro (robot description, xacro)
@@ -22,10 +22,9 @@
   <!-- Links: inertial,visual,collision -->
   <link name="base_human_link">
-    <inertial>
-      <!-- origin is relative -->
+    <!-- <inertial>
       <origin xyz="0 0 0.2" rpy="0 0 0"/>
       <mass value="5"/>
       <inertia ixx="5" ixy="0" ixz="0" iyy="5" iyz="0" izz="5"/>
-    </inertial>
+    </inertial> -->
     <visual>
       <geometry>
@@ -146,5 +145,5 @@
   </link>
   <joint name="body_bodyright_joint" type="fixed">
-      <origin xyz="0.0 -0.125 0" rpy="0 ${-90 * deg_to_rad} 0"/>
+    <origin xyz="0.0 -0.125 0" rpy="0 ${-90 * deg_to_rad} 0"/>
     <child link="bodyright_link"/>
     <parent link="body_link"/>
@@ -493,5 +492,5 @@
     <parent link="bodyright_link"/>
      <axis xyz="0 1 0"/>
-    <limit effort="1000.0" lower="-0.5" upper="0.5" velocity="0.5"/>
+    <limit effort="1000.0" lower="-0.6" upper="0.6" velocity="0.5"/>
   </joint>
   <link name="armright1_link">
@@ -522,5 +521,5 @@
     <parent link="shoulderright_link"/>
     <axis xyz="0 0 1"/>
-    <limit effort="1000.0" lower="-0.5" upper="0.5" velocity="0.5"/>
+    <limit effort="1000.0" lower="-0.6" upper="0.6" velocity="0.5"/>
     <!-- <calibration rising="0.0"/>
     <dynamics damping="0.0" friction="0.0"/>
@@ -579,5 +578,5 @@
     <parent link="armright1_link"/>
     <axis xyz="0 1 0"/>
-    <limit effort="1000.0" lower="-0.5" upper="0.5" velocity="0.5"/>
+    <limit effort="1000.0" lower="-0.6" upper="0.6" velocity="0.5"/>
   </joint>
   <link name="armleft2_link">
@@ -656,7 +655,7 @@
     </collision>
   </link>
-  <joint name="armright2_armright3_joint" type="fixed"> <!-- move from elbow down -->
+  <joint name="armright2_armright3_joint" type="revolute"> <!-- move from elbow down -->
       <axis xyz="1 1 1"/>
-      <limit effort="1000.0" lower="-0.5" upper="0.5" velocity="0.5"/>
+      <limit effort="1000.0" lower="-0.6" upper="0.6" velocity="0.5"/>
       <origin xyz="-0.065 0 0.11" rpy="0 ${-30 * deg_to_rad} 0"/>
     <child link="armright3_link"/>
@@ -871,5 +870,5 @@
   <child link="base_0"/>
   <origin xyz="0 0 0" rpy="0 0 -3.14" />
-  <axis xyz="0 0 1" />
+  <axis xyz="0 1 0" />
 </joint>
 <joint name="wr_j1" type="fixed"> <!--"continuous" -->
@@ -1352,4 +1351,14 @@
   </joint>
   <actuator name="motor4">
+    <hardwareInterface>hardware_interface/EffortJointInterface</hardwareInterface>
+    <mechanicalReduction>1</mechanicalReduction>
+  </actuator>
+</transmission>
+<transmission name="armright2_armright3_joint_tran">
+  <type>transmission_interface/SimpleTransmission</type>
+  <joint name="armright2_armright3_joint">
+    <hardwareInterface>hardware_interface/EffortJointInterface</hardwareInterface>
+  </joint>
+  <actuator name="motor5">
     <hardwareInterface>hardware_interface/EffortJointInterface</hardwareInterface>
     <mechanicalReduction>1</mechanicalReduction>

Commit message: adding costs and mln files

File: human_model_gazebo/urdf/human.xacro (robot description, xacro)
@@ -18,5 +18,23 @@
   <xacro:property name="board_width" value="0.3" />
   <material name="white">
-    <color rgba="0.1254 0.1254 0.1254 0.8"/>
+    <color rgba="0.45 0.45 0.45 1"/>
+  </material>
+  <material name="wood">
+    <color rgba="0.54509 0.2705 0.0745 1"/>
+  </material>
+  <material name="black">
+    <color rgba="1 1 1 1"/>
+  </material>
+  <material name="green">
+    <color rgba="0.95 0.95 0.95 1"/>
+  </material>
+  <material name="pink">
+    <color rgba="1 0.4 1 1"/>
+  </material>
+   <material name="orange">
+    <color rgba="0 1 1 1"/>
+  </material>
+   <material name="blue">
+    <color rgba="0 0 1 0.5"/>
   </material>
   <!-- Links: inertial,visual,collision -->
@@ -31,5 +49,5 @@
         <box size="${length} ${width} 0.04"/>
       </geometry>
-      <material name="white"/>
+      <material name="wood"/>
     </visual>
     <collision>
@@ -67,5 +85,5 @@
         <box size="${human_back_length} ${width} 0.04"/>
       </geometry>
-      <material name="white"/>
+      <material name="wood"/>
     </visual>
     <collision>
@@ -423,5 +441,5 @@
         <sphere radius="0.125"/>
       </geometry>
-      <material name="white"/>
+      <material name="black"/>
     </visual>
     <collision>
@@ -476,7 +494,7 @@
         <sphere radius="0.05"/>
       </geometry>
-      <material name="white"/>
-    </visual>
-    <material name="white"/>
+      <material name="green"/>
+    </visual>
+    <material name="green"/>
     <collision>
       <!-- origin is relative -->
@@ -505,5 +523,5 @@
         <cylinder radius="0.05" length="0.25"/>
       </geometry>
-      <material name="white"/>
+      <material name="green"/>
     </visual>
     <collision>
@@ -563,5 +581,5 @@
         <sphere radius="0.05"/>
       </geometry>
-      <material name="white"/>
+      <material name="green"/>
     </visual>
     <collision>
@@ -645,5 +663,5 @@
         <cylinder radius="0.05" length="0.2"/>
       </geometry>
-      <material name="white"/>
+      <material name="green"/>
     </visual>
     <collision>
@@ -655,5 +673,5 @@
     </collision>
   </link>
-  <joint name="armright2_armright3_joint" type="revolute"> <!-- move from elbow down -->
+  <joint name="armright2_armright3_joint" type="fixed"> <!-- move from elbow down -->
       <axis xyz="1 1 1"/>
       <limit effort="1000.0" lower="-0.6" upper="0.6" velocity="0.5"/>
@@ -669,10 +687,10 @@
       <inertia ixx="5" ixy="0" ixz="0" iyy="5" iyz="0" izz="5"/>
     </inertial>
-    <!-- <visual>
+    <visual>
       <geometry>
         <sphere radius="0.065"/>
       </geometry>
-      <material name="white"/>
-    </visual> -->
+      <material name="green"/>
+    </visual>
     <collision>
       <!-- origin is relative -->

File: human_model_gazebo/urdf/wheel.xacro (robot description, xacro)
@@ -5,5 +5,5 @@
   <xacro:property name="steer_velocity" value="5.0"/>
   <material name="gray">
-    <color rgba="0.1254 0.1254 0.1254 0.8"/>
+    <color rgba="0.54509 0.2705 0.0745 1"/>
   </material>
   <macro name="front_wheel" params="name parent radius thickness length width axel_offset right_left steer_height ">
